File: Hardware/Logger v2/Logger_v2.brd (EAGLE design)
At the start: 124.1 x 44.8 mm, 87 parts, among them IC1 24AA256SN, J6 5.5x2.1mm Barrel, Q5 4.3A/20V/54mΩ, Q6 4.3A/20V/54mΩ, Q7 4.3A/20V/54mΩ, Q8 220mA/50V/3.5Ω, Q9 220mA/50V/3.5Ω, U1 ATSAMD21G-A, U3 915MHz, U4 SX1509

Commit message: PCB Major Issues Fixed
All major issues on the PCB are fixed and only remaining problems are with solder mask spacing. Ready for final functional check
Parts:
- removed S3: MOMENTARY-SWITCH-SPST-SMD-5.2MM, SparkFun-Switches:TACTILE_SWITCH_SMD_5.2MM
- added U$1: SKRPABE010, Custom:SKRPABE010_(SWITCH)
- BT1: value (none) -> LINX-BAT-HLD-012-SMT-OTL; device SparkFun-Batteries:BATTCON_12MM -> awickert:LINX_BAT-HLD-012-SMT
- S2: value MOMENTARY-SWITCH-SPST-SMD-5.2MM -> SKRPABE010; device SparkFun-Switches:TACTILE_SWITCH_SMD_5.2MM -> Custom:SKRPABE010_(SWITCH)
- moved F2 2.01 mm to (74.6, 21.0)
- moved X1 0.95 mm to (118.4, 5.08)
- moved S2 0.79 mm to (4.45, 5.71)
- moved D1 0.32 mm to (77.9, 27.8)
- moved D2 0.32 mm to (75.7, 27.8)
- moved D3 0.32 mm to (73.5, 27.8)
- moved U3 0.32 mm to (105.1, 11.4)
- moved J4 0.24 mm to (115.3, 24.4)
- moved J6 0.24 mm to (112.8, 35.6)
- moved R23 0.24 mm to (77.9, 30.9)
- moved R24 0.24 mm to (75.7, 30.9)
- moved R25 0.24 mm to (73.5, 30.9)
- moved C6 0.16 mm to (54.1, 33.0)
- moved C7 0.16 mm to (49.7, 25.6)
- moved C5 0.16 mm to (54.1, 34.8)
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Connections:
- net GND: now also S2.P$3, S2.P$4, U$1.P$1, U$1.P$2; no longer S2.3, S3.1
- net N$31: now also BT1.POWER0, BT1.POWER1; no longer BT1.PWR@1
- net N$5: now also S2.P$1, S2.P$2; no longer S2.1
- net RST: now also U$1.P$3, U$1.P$4; no longer S3.3
Routing:
- net RST: track 76.0 -> 89.6 mm
- net 3.3V: track 372.0 -> 383.4 mm
- net MUX_INT: track 20.4 -> 25.7 mm
- net N$5: track 64.9 -> 70.1 mm
- net EXT_5V: track 108.8 -> 112.4 mm
- net GND: track 690.0 -> 692.4 mm
- net MISO: track 154.1 -> 155.7 mm
- net BATT+: track 155.4 -> 153.9 mm
- net N$18: track 1.63 -> 2.90 mm
- net USB_D-: track 62.3 -> 61.2 mm
- net SCL: track 143.4 -> 142.4 mm
- net RADIO_CS: track 59.5 -> 58.6 mm
- net USB_HOST_EN: track 53.3 -> 52.4 mm
- net EXT_3.3V: track 143.5 -> 144.5 mm
- net EXT_INT: track 28.2 -> 29.0 mm
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Other:
- board size 124.1 x 44.8 mm -> 124.1 x 45.3 mm
- board text added: "3V3"
- board text added: "5V"
- board text added: "A0"
- board text added: "A1"
- board text added: "A10"
- board text added: "A11"
- board text added: "A2"
- board text added: "A3"
- board text added: "A4"
- board text added: "A5"
- board text added: "A6"
- board text added: "A7"
- board text added: "A8"
- board text added: "A9"
- board text added: "CS2"
- board text added: "D0"
- board text added: "D1"
- board text added: "D2"
- board text added: "D3"
- board text added: "D6"
- board text added: "DI"
- board text added: "DO"
- board text added: "GND"
- board text added: "I2C"
- board text added: "INT1"
- board text added: "ISP"
- board text added: "LOG"
- board text added: "RESET"
- board text added: "RX"
- board text added: "SCK"
- board text added: "SCL"
- board text added: "SDA"
- board text added: "SPI"
- board text added: "TX"
- board text added: "VIN"

Commit message: Final PCB Logger Design
The final design iteration for the logger PCB
Parts:
- C18: value (none) -> .1uF
- C7: value (none) -> 1uF
- C8, C9: value (none) -> 12nF
- R13, R14, R16, R17: value (none) -> FB
- R23, R24, R25: value (none) -> 330
- R44, R45, R46, R47: value (none) -> 10k
- U3: device SparkFun-RF:RFM69CW-XXXS2 -> SparkFun-RF:RFM69HCW-XXXS2
- moved J6 1.59 mm to (111.2, 35.6)
- moved IC1 1.27 mm to (63.5, 11.4)
- moved U3 0.56 mm to (104.7, 11.8), turned to 0 degrees
Connections:
- removed net EEPROM_WP: IC1.7
- net 3.3V: now also U3.13; no longer U3.2
- net GND: now also IC1.7, U1.35, U3.1, U3.10, U3.8; no longer U3.14, U3.3
- net MISO: now also U3.2; no longer U3.8
- net MOSI: now also U3.3; no longer U3.5
- net N$28: now also U3.9; no longer U3.1
- net RADIO_CS: now also U3.5; no longer U3.7
- net RADIO_INT: now also U3.14; no longer U3.9
- net SCK: now also U3.4; no longer U3.6
Routing:
- net GND: track 692.4 -> 727.4 mm, vias 9 -> 14
- net RADIO_INT: track 48.5 -> 64.0 mm
- net MOSI: track 171.9 -> 158.2 mm
- net SCK: track 173.0 -> 160.2 mm
- net BATT+: track 153.9 -> 150.7 mm
- net RADIO_CS: track 58.6 -> 55.7 mm
- net USB_HOST_EN: track 52.4 -> 53.9 mm
- net 3.3V: track 383.4 -> 381.9 mm, vias 14 -> 15
- net SCL: track 142.4 -> 143.7 mm
